Commit message: refactor: Add camera and lidar to robot model

File: src/my_robot/urdf/my_robot.xacro (robot description, xacro)
@@ -117,3 +117,61 @@
     <dynamics damping="1.0" friction="1.0"/>
   </joint>
+  <link name='camera'>
+   <inertial>
+      <mass value="0.1"/>
+      <origin xyz="0 0 0" rpy="0 0 0"/>
+      <inertia
+          ixx="1e-6" ixy="0" ixz="0"
+          iyy="1e-6" iyz="0"
+          izz="1e-6"
+      />
+    </inertial>
+    <collision name='camera_collision'>
+       <origin xyz="0 0 0" rpy="0 0 0"/>
+       <geometry>
+         <box size="0.05 0.05 0.05"/>
+       </geometry>
+    </collision>
+    <visual name='camera_visual'>
+      <origin xyz="0 0 0" rpy="0 0 0"/>
+      <geometry>
+        <box size="0.05 0.05 0.05"/>
+      </geometry>
+    </visual>
+  </link>
+  <joint name="camera_joint" type="fixed">
+	<origin xyz="0.2 0 0" rpy="0 0 0" />
+	<child link="camera" />
+	<parent link="chassis" />
+	<axis xyz="0 1 0" />
+  </joint>
+  <link name='hokuyo'>
+   <inertial>
+      <mass value="1e-5"/>
+      <origin xyz="0 0 0" rpy="0 0 0"/>
+      <inertia
+          ixx="1e-6" ixy="0" ixz="0"
+          iyy="1e-6" iyz="0"
+          izz="1e-6"
+      />
+    </inertial>
+    <collision name='hokuyo_collision'>
+       <origin xyz="0 0 0" rpy="0 0 0"/>
+       <geometry>
+         <box size="0.1 0.1 0.1"/>
+       </geometry>
+    </collision>
+    <visual name='hokuyo_visual'>
+       <origin xyz="0 0 0" rpy="0 0 0"/>
+       <geometry>
+         <mesh filename = "package://my_robot/meshes/hokuyo.dae"/>
+       </geometry>
+    </visual>
+  </link>
+  <joint name="hokuyo" type="fixed">
+	<origin xyz="0.15 0 0.1" rpy="0 0 0" />
+	<child link="hokuyo" />
+	<parent link="chassis" />
+        <axis xyz="0 1 0" />
+  </joint>
 </robot>

Commit message: refactor: Change robot dimensions and set colour

File: src/my_robot/urdf/my_robot.xacro (robot description, xacro)
@@ -2,4 +2,17 @@
 <robot name="my_robot" xmlns:xacro="http://www.ros.org/wiki/xacro">
   <xacro:include filename="$(find my_robot)/urdf/my_robot.gazebo" />
+  <xacro:include filename="$(find my_robot)/urdf/materials.xacro" />
+  <gazebo reference = 'chassis'>
+    <material> Gazebo/Indigo </material>
+  </gazebo>
+  <gazebo reference = 'left_wheel'>
+    <material> Gazebo/Yellow </material>
+  </gazebo>
+  <gazebo reference = 'right_wheel'>
+    <material> Gazebo/Yellow </material>
+  </gazebo>
+  <gazebo reference = 'camera'>
+    <material> Gazebo/Green </material>
+  </gazebo>
   <link name="robot_footprint"></link>
   <joint name="robot_footprint_joint" type="fixed">
@@ -22,5 +35,5 @@
       <origin xyz="0 0 0" rpy=" 0 0 0"/>
       <geometry>
-        <box size=".4 .2 .1"/>
+        <box size=".4 .3 .175"/>
       </geometry>
     </collision>
@@ -28,29 +41,30 @@
       <origin xyz="0 0 0" rpy=" 0 0 0"/>
       <geometry>
-        <box size=".4 .2 .1"/>
+        <box size=".4 .3 .175"/>
       </geometry>
+    <material name="indigo"/>
     </visual>
     <collision name='back_caster_collision'>
-      <origin xyz="-0.15 0 -0.05" rpy=" 0 0 0"/>
+      <origin xyz="-0.125 0 -0.075" rpy=" 0 0 0"/>
       <geometry>
-        <sphere radius="0.0499"/>
+        <sphere radius="0.07499"/>
       </geometry>
     </collision>
     <visual name='back_caster_visual'>
-      <origin xyz="-0.15 0 -0.05" rpy=" 0 0 0"/>
+      <origin xyz="-0.125 0 -0.075" rpy=" 0 0 0"/>
       <geometry>
-        <sphere radius="0.05"/>
+        <sphere radius="0.075"/>
       </geometry>
     </visual>
     <collision name='front_caster_collision'>
-      <origin xyz="0.15 0 -0.05" rpy=" 0 0 0"/>
+      <origin xyz="0.125 0 -0.075" rpy=" 0 0 0"/>
       <geometry>
-        <sphere radius="0.0499"/>
+        <sphere radius="0.07499"/>
       </geometry>
     </collision>
     <visual name='front_caster_visual'>
-      <origin xyz="0.15 0 -0.05" rpy=" 0 0 0"/>
+      <origin xyz="0.125 0 -0.075" rpy=" 0 0 0"/>
       <geometry>
-        <sphere radius="0.05"/>
+        <sphere radius="0.075"/>
       </geometry>
     </visual>
@@ -69,5 +83,5 @@
        <origin xyz="0 0 0" rpy="0 1.5707 1.5707"/>
        <geometry>
-         <cylinder length="0.05" radius="0.1"/>
+         <cylinder length="0.07" radius="0.15"/>
        </geometry>
     </collision>
@@ -75,10 +89,11 @@
       <origin xyz="0 0 0" rpy="0 1.5707 1.5707"/>
       <geometry>
-        <cylinder length="0.05" radius="0.1"/>
+        <cylinder length="0.07" radius="0.15"/>
       </geometry>
+    <material name="yellow"/>
     </visual>
   </link>
   <joint type="continuous" name="left_wheel_hinge">
-    <origin xyz="0 0.15 0" rpy="0 0 0"/>
+    <origin xyz="0 0.25 0" rpy="0 0 0"/>
     <child link="left_wheel"/>
     <parent link="chassis"/>
@@ -87,5 +102,5 @@
     <dynamics damping="1.0" friction="1.0"/>
   </joint>
-  <link name='rigth_wheel'>
+  <link name='right_wheel'>
    <inertial>
       <mass value="5.0"/>
@@ -100,5 +115,5 @@
        <origin xyz="0 0 0" rpy="0 1.5707 1.5707"/>
        <geometry>
-         <cylinder length="0.05" radius="0.1"/>
+         <cylinder length="0.07" radius="0.15"/>
        </geometry>
     </collision>
@@ -106,11 +121,12 @@
       <origin xyz="0 0 0" rpy="0 1.5707 1.5707"/>
       <geometry>
-        <cylinder length="0.05" radius="0.1"/>
+        <cylinder length="0.07" radius="0.15"/>
       </geometry>
+    <material name="yellow"/>
     </visual>
   </link>
   <joint type="continuous" name="right_wheel_hinge">
-    <origin xyz="0 -0.15 0" rpy="0 0 0"/>
-    <child link="rigth_wheel"/>
+    <origin xyz="0 -0.25 0" rpy="0 0 0"/>
+    <child link="right_wheel"/>
     <parent link="chassis"/>
     <axis xyz="0 1 0" rpy="0 0 0"/>
@@ -139,4 +155,5 @@
         <box size="0.05 0.05 0.05"/>
       </geometry>
+    <material name="green"/>
     </visual>
   </link>

Commit message: refactor: Modify robot model

File: src/my_robot/urdf/my_robot.xacro (robot description, xacro)
@@ -32,8 +32,8 @@
       />
     </inertial>
-    <collision name='collision'>
+    <collision name='chassis_collision'>
       <origin xyz="0 0 0" rpy=" 0 0 0"/>
       <geometry>
-        <box size=".4 .3 .175"/>
+        <box size=".4 .3 .17"/>
       </geometry>
     </collision>
@@ -41,5 +41,5 @@
       <origin xyz="0 0 0" rpy=" 0 0 0"/>
       <geometry>
-        <box size=".4 .3 .175"/>
+        <box size=".4 .3 .17"/>
       </geometry>
     <material name="indigo"/>
@@ -48,5 +48,5 @@
       <origin xyz="-0.125 0 -0.075" rpy=" 0 0 0"/>
       <geometry>
-        <sphere radius="0.07499"/>
+        <sphere radius="0.0749"/>
       </geometry>
     </collision>
@@ -60,5 +60,5 @@
       <origin xyz="0.125 0 -0.075" rpy=" 0 0 0"/>
       <geometry>
-        <sphere radius="0.07499"/>
+        <sphere radius="0.0749"/>
       </geometry>
     </collision>

Commit message: refactor: Modify my robot model and adjust plugin file

File: src/my_robot/urdf/my_robot.xacro (robot description, xacro)
@@ -35,5 +35,5 @@
       <origin xyz="0 0 0" rpy=" 0 0 0"/>
       <geometry>
-        <box size=".4 .3 .17"/>
+        <box size=".6 .3 .17"/>
       </geometry>
     </collision>
@@ -41,10 +41,10 @@
       <origin xyz="0 0 0" rpy=" 0 0 0"/>
       <geometry>
-        <box size=".4 .3 .17"/>
+        <box size=".6 .3 .17"/>
       </geometry>
     <material name="indigo"/>
     </visual>
     <collision name='back_caster_collision'>
-      <origin xyz="-0.125 0 -0.075" rpy=" 0 0 0"/>
+      <origin xyz="-0.225 0 -0.075" rpy=" 0 0 0"/>
       <geometry>
         <sphere radius="0.0749"/>
@@ -52,5 +52,5 @@
     </collision>
     <visual name='back_caster_visual'>
-      <origin xyz="-0.125 0 -0.075" rpy=" 0 0 0"/>
+      <origin xyz="-0.225 0 -0.075" rpy=" 0 0 0"/>
       <geometry>
         <sphere radius="0.075"/>
@@ -58,5 +58,5 @@
     </visual>
     <collision name='front_caster_collision'>
-      <origin xyz="0.125 0 -0.075" rpy=" 0 0 0"/>
+      <origin xyz="0.225 0 -0.075" rpy=" 0 0 0"/>
       <geometry>
         <sphere radius="0.0749"/>
@@ -64,5 +64,5 @@
     </collision>
     <visual name='front_caster_visual'>
-      <origin xyz="0.125 0 -0.075" rpy=" 0 0 0"/>
+      <origin xyz="0.225 0 -0.075" rpy=" 0 0 0"/>
       <geometry>
         <sphere radius="0.075"/>
@@ -83,5 +83,5 @@
        <origin xyz="0 0 0" rpy="0 1.5707 1.5707"/>
        <geometry>
-         <cylinder length="0.07" radius="0.15"/>
+         <cylinder length="0.075" radius="0.15"/>
        </geometry>
     </collision>
@@ -89,5 +89,5 @@
       <origin xyz="0 0 0" rpy="0 1.5707 1.5707"/>
       <geometry>
-        <cylinder length="0.07" radius="0.15"/>
+        <cylinder length="0.075" radius="0.15"/>
       </geometry>
     <material name="yellow"/>
@@ -115,5 +115,5 @@
        <origin xyz="0 0 0" rpy="0 1.5707 1.5707"/>
        <geometry>
-         <cylinder length="0.07" radius="0.15"/>
+         <cylinder length="0.075" radius="0.15"/>
        </geometry>
     </collision>
@@ -121,5 +121,5 @@
       <origin xyz="0 0 0" rpy="0 1.5707 1.5707"/>
       <geometry>
-        <cylinder length="0.07" radius="0.15"/>
+        <cylinder length="0.075" radius="0.15"/>
       </geometry>
     <material name="yellow"/>
@@ -159,5 +159,5 @@
   </link>
   <joint name="camera_joint" type="fixed">
-	<origin xyz="0.2 0 0" rpy="0 0 0" />
+	<origin xyz="0.3 0 0" rpy="0 0 0" />
 	<child link="camera" />
 	<parent link="chassis" />
@@ -188,5 +188,5 @@
   </link>
   <joint name="hokuyo" type="fixed">
-	<origin xyz="0.15 0 0.1" rpy="0 0 0" />
+	<origin xyz="0.25 0 0.15" rpy="0 0 0" />
 	<child link="hokuyo" />
 	<parent link="chassis" />
